Commit message: refactor: robot configuration and launch files; add integration tests and update dependencies

File: my_robot_description/urdf/base/base.gazebo.xacro (robot description, xacro)
@@ -3,5 +3,5 @@
   <!-- Gazebo material for chassis -->
   <gazebo reference="chassis">
-    <material>Gazebo/Grey</material>
+    <material>Gazebo/Blue</material>
   </gazebo>
   <!-- Gazebo material for casters -->
@@ -13,9 +13,7 @@
   </gazebo>
   <!-- ros2_control Gazebo plugin: bridges ros2_control to Gazebo joints -->
+  <!-- controller_manager is launched explicitly and owns controllers.yaml -->
   <gazebo>
-    <plugin name="gz_ros2_control::GazeboSimROS2ControlPlugin" filename="libgz_ros2_control-system">
-      <parameters>$(find my_robot_description)/config/controllers.yaml</parameters>
-      <parameters>$(find my_robot_description)/config/joint_limits.yaml</parameters>
-    </plugin>
+    <plugin name="gz_ros2_control::GazeboSimROS2ControlPlugin" filename="libgz_ros2_control-system"/>
   </gazebo>
 </robot>

File: my_robot_description/urdf/base/base.ros2_control.xacro (robot description, xacro)
@@ -1,15 +1,22 @@
 <?xml version="1.0"?>
 <robot xmlns:xacro="http://www.ros.org/wiki/xacro" name="base_ros2_control">
-  <ros2_control name="my_robot" type="system">
+  <xacro:arg name="hardware_plugin" default="mock_components/GenericSystem"/>
+  <ros2_control name="my_robot_hardware_interface" type="system">
     <hardware>
-      <plugin>gazebo_ros2_control/GazeboSystem</plugin>
+      <plugin>$(arg hardware_plugin)</plugin>
     </hardware>
     <joint name="chassis_to_left_wheel_joint">
-      <command_interface name="velocity"/>
+      <command_interface name="velocity">
+        <param name="max_velocity">1.0</param>
+        <param name="min_velocity">-1.0</param>
+      </command_interface>
       <state_interface name="velocity"/>
       <state_interface name="position"/>
     </joint>
     <joint name="chassis_to_right_wheel_joint">
-      <command_interface name="velocity"/>
+      <command_interface name="velocity">
+        <param name="max_velocity">1.0</param>
+        <param name="min_velocity">-1.0</param>
+      </command_interface>
       <state_interface name="velocity"/>
       <state_interface name="position"/>

File: my_robot_description/urdf/my_robot.urdf.xacro (robot description, xacro)
@@ -6,4 +6,5 @@
   <xacro:include filename="$(find my_robot_description)/urdf/base/base.xacro"/>
   <xacro:include filename="$(find my_robot_description)/urdf/base/base.gazebo.xacro"/>
+  <!-- Robot Controls -->
   <xacro:include filename="$(find my_robot_description)/urdf/base/base.ros2_control.xacro"/>
   <!-- Driven wheel macro -->
