Commit message: refactor: URDF and Xacro files to replace 'lidar' with 'hokuyo_lidar'

File: src/robot_description/urdf/common/robot_properties.xacro (robot description, xacro)
@@ -14,8 +14,4 @@
   <xacro:property name="caster_mass" value="0.5"/>
   <xacro:property name="caster_inset" value="0.02"/>
-  <!-- Lidar dimensions (cylinder mounted upright) -->
-  <xacro:property name="lidar_radius" value="0.05"/>
-  <xacro:property name="lidar_height" value="0.07"/>
-  <xacro:property name="lidar_mass" value="0.2"/>
   <!-- Camera dimensions (box: x=depth, y=width, z=height) -->
   <xacro:property name="camera_size_x" value="0.03"/>

File: src/robot_description/urdf/sensors/camera.gazebo.xacro (robot description, xacro)
@@ -2,5 +2,5 @@
 <robot xmlns:xacro="http://www.ros.org/wiki/xacro" name="camera_gazebo">
   <gazebo reference="camera">
-    <sensor name="camera" type="camera">
+    <sensor name="rgb_camera" type="camera">
       <pose>0 0 0 0 0 0</pose>
       <topic>/camera/image_raw</topic>
@@ -18,5 +18,5 @@
       </camera>
     </sensor>
-    <material>Gazebo/Blue</material>
+    <material>Gazebo/Red</material>
   </gazebo>
 </robot>

File: src/robot_description/urdf/sensors/lidar.gazebo.xacro (robot description, xacro)
@@ -1,5 +1,5 @@
 <?xml version="1.0"?>
 <robot xmlns:xacro="http://www.ros.org/wiki/xacro" name="lidar_gazebo">
-  <gazebo reference="lidar">
+  <gazebo reference="hokuyo_lidar">
     <sensor name="gpu_lidar" type="gpu_lidar">
       <pose>0 0 0 0 0 0</pose>
@@ -27,5 +27,4 @@
       </lidar>
     </sensor>
-    <material>Gazebo/Red</material>
   </gazebo>
 </robot>

File: src/robot_description/urdf/sensors/lidar.xacro (robot description, xacro)
@@ -1,42 +1,28 @@
 <?xml version="1.0"?>
 <robot xmlns:xacro="http://www.ros.org/wiki/xacro" name="lidar">
-  <!-- Lidar link: frame at the cylinder's geometric center -->
-  <link name="lidar">
+  <link name="hokuyo_lidar">
     <inertial>
-      <mass value="${lidar_mass}"/>
+      <mass value="1e-5"/>
       <origin xyz="0 0 0" rpy="0 0 0"/>
-      <inertia
-          ixx="${lidar_mass * (3*lidar_radius**2 + lidar_height**2) / 12}"
-          ixy="0"
-          ixz="0"
-          iyy="${lidar_mass * (3*lidar_radius**2 + lidar_height**2) / 12}"
-          iyz="0"
-          izz="${lidar_mass * lidar_radius**2 / 2}"/>
+      <inertia ixx="1e-6" ixy="0" ixz="0" iyy="1e-6" iyz="0" izz="1e-6"/>
     </inertial>
     <visual>
       <origin xyz="0 0 0" rpy="0 0 0"/>
       <geometry>
-        <cylinder radius="${lidar_radius}" length="${lidar_height}"/>
+        <mesh filename="package://robot_description/meshes/sensors/hokuyo_lidar.dae"/>
       </geometry>
-      <material name="red">
-        <color rgba="1.0 0.0 0.0 1.0"/>
-      </material>
     </visual>
     <collision>
       <origin xyz="0 0 0" rpy="0 0 0"/>
       <geometry>
-        <cylinder radius="${lidar_radius}" length="${lidar_height}"/>
+        <box size="0.05 0.05 0.07"/>
       </geometry>
     </collision>
   </link>
-  <!--
-    Lidar joint: mount on top of chassis.
-      z-offset = chassis_height/2 + lidar_height/2
-        (lidar bottom flush with chassis top)
-  -->
-  <joint name="chassis_to_lidar_joint" type="fixed">
-    <origin xyz="0 0 ${chassis_height/2 + lidar_height/2}" rpy="0 0 0"/>
+  <joint name="chassis_to_hokuyo_lidar_joint" type="fixed">
+    <axis xyz="0 1 0"/>
+    <origin xyz="0.15 0 ${chassis_height/2}" rpy="0 0 0"/>
     <parent link="chassis"/>
-    <child link="lidar"/>
+    <child link="hokuyo_lidar"/>
   </joint>
 </robot>

File: src/robot_description/urdf/wheels/caster.xacro (robot description, xacro)
@@ -27,5 +27,5 @@
         <origin xyz="0 0 0" rpy="0 0 0"/>
         <geometry>
-          <sphere radius="${caster_radius}"/>
+          <sphere radius="${caster_radius - 0.0001}"/>
         </geometry>
       </collision>

File: src/robot_description/urdf/wheels/wheel.gazebo.xacro (robot description, xacro)
@@ -3,10 +3,10 @@
   <!-- Wheel material and friction -->
   <gazebo reference="left_wheel">
-    <material>Gazebo/Black</material>
+    <material>Gazebo/Green</material>
     <mu1>0.8</mu1>
     <mu2>0.8</mu2>
   </gazebo>
   <gazebo reference="right_wheel">
-    <material>Gazebo/Black</material>
+    <material>Gazebo/Green</material>
     <mu1>0.8</mu1>
     <mu2>0.8</mu2>
