Commit message: chore: tune to the correct lidar height

File: src/robot_description/urdf/sensors/lidar.xacro (robot description, xacro)
@@ -22,5 +22,5 @@
   <joint name="chassis_to_hokuyo_lidar_joint" type="fixed">
     <axis xyz="0 1 0"/>
-    <origin xyz="0.15 0 ${chassis_height/2}" rpy="0 0 0"/>
+    <origin xyz="0.15 0 ${chassis_height/2 + 0.035}" rpy="0 0 0"/>
     <parent link="chassis"/>
     <child link="hokuyo_lidar"/>
