Commit message: chore: add coloring to robot parts
Co-authored-by: Copilot <copilot@github.com>

File: src/robot_description/urdf/base/base.xacro (robot description, xacro)
@@ -28,6 +28,6 @@
         <box size="${chassis_length} ${chassis_width} ${chassis_height}"/>
       </geometry>
-      <material name="steel">
-        <color rgba="0.5 0.5 0.5 1.0"/>
+      <material name="blue">
+        <color rgba="0.0 0.0 1.0 1.0"/>
       </material>
     </visual>

File: src/robot_description/urdf/sensors/camera.xacro (robot description, xacro)
@@ -19,6 +19,6 @@
         <box size="${camera_size_x} ${camera_size_y} ${camera_size_z}"/>
       </geometry>
-      <material name="blue">
-        <color rgba="0.0 0.0 1.0 1.0"/>
+      <material name="red">
+        <color rgba="1.0 0.0 0.0 1.0"/>
       </material>
     </visual>
