Commit message: feat: ported apartment model from old repo into this one to have an all in one solution

File: src/robot_description/urdf/base/base.xacro (robot description, xacro)
@@ -6,5 +6,5 @@
   <!-- Lift chassis frame to wheel-axle height + half chassis -->
   <joint name="robot_footprint_to_chassis_joint" type="fixed">
-    <origin xyz="0 0 ${chassis_z}" rpy="0 0 0"/>
+    <origin xyz="0 1 ${chassis_z}" rpy="0 0 0"/>
     <parent link="robot_footprint"/>
     <child link="chassis"/>

File: src/robot_description/urdf/robot.gazebo.urdf.xacro (robot description, xacro)
@@ -5,5 +5,5 @@
   gz_ros2_control, avoiding the parameter-file forwarding bug in
   gz_ros2_control 1.2.17 (ros-controls/gz_ros2_control#512).
-  Not used for display or real-hardware launches — those use robot.urdf.xacro
+  Not used for display only or real-hardware launches — those use robot.urdf.xacro
   with mock_components/GenericSystem or the real hardware plugin.
 -->

Commit message: chore: get rid of dead code

File: src/robot_description/urdf/base/base.xacro (robot description, xacro)
@@ -40,3 +40,13 @@
   <xacro:caster prefix="front" x_offset="${chassis_length/2 - caster_radius - caster_inset}"/>
   <xacro:caster prefix="back" x_offset="${-(chassis_length/2 - caster_radius - caster_inset)}"/>
+  <!-- Gazebo materials -->
+  <gazebo reference="chassis">
+    <material>Gazebo/Blue</material>
+  </gazebo>
+  <gazebo reference="front_caster">
+    <material>Gazebo/DarkGrey</material>
+  </gazebo>
+  <gazebo reference="back_caster">
+    <material>Gazebo/DarkGrey</material>
+  </gazebo>
 </robot>

File: src/robot_description/urdf/robot.urdf.xacro (robot description, xacro)
@@ -22,3 +22,9 @@
     </plugin>
   </gazebo>
+  <!-- Gazebo sensor rendering pipeline -->
+  <gazebo>
+    <plugin filename="gz-sim-sensors-system" name="gz::sim::systems::Sensors">
+      <render_engine>ogre2</render_engine>
+    </plugin>
+  </gazebo>
 </robot>

File: src/robot_description/urdf/sensors/camera.xacro (robot description, xacro)
@@ -45,3 +45,24 @@
     <child link="camera_optical_frame"/>
   </joint>
+  <!-- Gazebo RGB camera sensor -->
+  <gazebo reference="camera">
+    <sensor name="rgb_camera" type="camera">
+      <pose>0 0 0 0 0 0</pose>
+      <gz_frame_id>camera_optical_frame</gz_frame_id>
+      <topic>/camera/rgb/image_raw</topic>
+      <update_rate>30</update_rate>
+      <camera>
+        <image>
+          <width>640</width>
+          <height>480</height>
+          <format>R8G8B8</format>
+        </image>
+        <clip>
+          <near>0.01</near>
+          <far>100.0</far>
+        </clip>
+      </camera>
+    </sensor>
+    <material>Gazebo/Red</material>
+  </gazebo>
 </robot>

File: src/robot_description/urdf/sensors/lidar.xacro (robot description, xacro)
@@ -26,3 +26,32 @@
     <child link="hokuyo_lidar"/>
   </joint>
+  <!-- Gazebo GPU lidar sensor -->
+  <gazebo reference="hokuyo_lidar">
+    <sensor name="gpu_lidar" type="gpu_lidar">
+      <pose>0 0 0 0 0 0</pose>
+      <gz_frame_id>hokuyo_lidar</gz_frame_id>
+      <topic>/scan</topic>
+      <update_rate>20</update_rate>
+      <lidar>
+        <scan>
+          <horizontal>
+            <samples>360</samples>
+            <resolution>1.0</resolution>
+            <min_angle>0.0</min_angle>
+            <max_angle>6.28318530718</max_angle>
+          </horizontal>
+        </scan>
+        <range>
+          <min>0.1</min>
+          <max>10.0</max>
+          <resolution>0.01</resolution>
+        </range>
+        <noise>
+          <type>gaussian</type>
+          <mean>0.0</mean>
+          <stddev>0.01</stddev>
+        </noise>
+      </lidar>
+    </sensor>
+  </gazebo>
 </robot>

File: src/robot_description/urdf/wheels/wheel.xacro (robot description, xacro)
@@ -52,3 +52,14 @@
     </joint>
   </xacro:macro>
+  <!-- Gazebo wheel materials and friction -->
+  <gazebo reference="left_wheel">
+    <material>Gazebo/Green</material>
+    <mu1>0.8</mu1>
+    <mu2>0.8</mu2>
+  </gazebo>
+  <gazebo reference="right_wheel">
+    <material>Gazebo/Green</material>
+    <mu1>0.8</mu1>
+    <mu2>0.8</mu2>
+  </gazebo>
 </robot>

Commit message: chore: revert offset from footprint to chassis

File: src/robot_description/urdf/base/base.xacro (robot description, xacro)
@@ -6,5 +6,5 @@
   <!-- Lift chassis frame to wheel-axle height + half chassis -->
   <joint name="robot_footprint_to_chassis_joint" type="fixed">
-    <origin xyz="0 1 ${chassis_z}" rpy="0 0 0"/>
+    <origin xyz="0 0 ${chassis_z}" rpy="0 0 0"/>
     <parent link="robot_footprint"/>
     <child link="chassis"/>
