Commit message: refactor: update robot configuration and launch files for diff_drive_controller integration

File: src/robot_description/urdf/base/base.gazebo.xacro (robot description, xacro)
@@ -13,7 +13,6 @@
   </gazebo>
   <!-- ros2_control Gazebo plugin: bridges ros2_control to Gazebo joints -->
-  <!-- controller_manager is launched explicitly and owns controllers.yaml -->
   <gazebo>
-    <plugin name="gz_ros2_control::GazeboSimROS2ControlPlugin" filename="libgz_ros2_control-system">
+    <plugin name="gz_ros2_control::GazeboSimROS2ControlPlugin" filename="gz_ros2_control-system">
       <parameters>$(find robot_description)/config/controllers.yaml</parameters>
     </plugin>

File: src/robot_description/urdf/base/base.xacro (robot description, xacro)
@@ -28,7 +28,5 @@
         <box size="${chassis_length} ${chassis_width} ${chassis_height}"/>
       </geometry>
-      <material name="blue">
-        <color rgba="0.0 0.0 1.0 1.0"/>
-      </material>
+      <material name="blue" />
     </visual>
     <collision>

File: src/robot_description/urdf/common/robot_properties.xacro (robot description, xacro)
@@ -22,3 +22,16 @@
   <!-- chassis frame sits at wheel-axle level, so wheels mount at chassis bottom -->
   <xacro:property name="chassis_z" value="${wheel_radius + chassis_height/2}"/>
+  <!-- RViz Colors -->
+  <material name="blue">
+    <color rgba="0.0 0.0 1.0 1.0"/>
+  </material>
+  <material name="red">
+    <color rgba="1.0 0.0 0.0 1.0"/>
+  </material>
+  <material name="black">
+    <color rgba="0.1 0.1 0.1 1.0"/>
+  </material>
+  <material name="grey">
+    <color rgba="0.3 0.3 0.3 1.0"/>
+  </material>
 </robot>

File: src/robot_description/urdf/sensors/camera.xacro (robot description, xacro)
@@ -19,7 +19,5 @@
         <box size="${camera_size_x} ${camera_size_y} ${camera_size_z}"/>
       </geometry>
-      <material name="red">
-        <color rgba="1.0 0.0 0.0 1.0"/>
-      </material>
+      <material name="red" />
     </visual>
     <collision>

File: src/robot_description/urdf/wheels/caster.xacro (robot description, xacro)
@@ -20,7 +20,5 @@
           <sphere radius="${caster_radius}"/>
         </geometry>
-        <material name="grey">
-          <color rgba="0.3 0.3 0.3 1.0"/>
-        </material>
+        <material name="grey" />
       </visual>
       <collision>

File: src/robot_description/urdf/wheels/wheel.xacro (robot description, xacro)
@@ -27,7 +27,5 @@
           <cylinder radius="${wheel_radius}" length="${wheel_length}"/>
         </geometry>
-        <material name="black">
-          <color rgba="0.1 0.1 0.1 1.0"/>
-        </material>
+        <material name="black" />
       </visual>
       <collision>
@@ -50,4 +48,6 @@
       <child link="${prefix}_wheel"/>
       <axis xyz="0 1 0"/>
+      <limit effort="10.0" velocity="10.0"/>   <!-- Nm and rad/s — used by ros2_control -->
+      <dynamics damping="0.1" friction="0.1"/> <!-- optional; used by sim and fake hardware -->
     </joint>
   </xacro:macro>
